File: Attenuator/DIY Pi attenuator/DIY Pi attenuator.kicad_sch (KiCad schematic)
At the start: 25 parts, among them U2 DPDT_switch, U3 DPDT_switch

Commit message: Pi attenuator Schematic
Parts:
- removed R6: (no value), symbol Device:R
- added R19, R20, R21, R22, R23, R24, R25, R26, R27, R28, R29, R3, R30, R31, R32, R33, R34, R35, R36: R, symbol Device:R
- added U4: DPDT_switch, symbol Custom:DPDT_switch
- C1, C2: value (none) -> C
- Input1: value (none) -> Conn_Coaxial
- R1: renamed from R2; value (none) -> R
- R2: renamed from R1; value (none) -> R
- R4: renamed from R3; value (none) -> R
- R5: value (none) -> R
- R6: renamed from R4; value (none) -> R
- U2: value DPDT_switch -> (none)
Connections:
- net Earth: now also R13.2, R14.2, R5.2, R22.2, R23.2, R24.2, R31.2, R32.2, R33.2; no longer R10.2, R16.2, R9.2
- net at R11.1, R12.1: now also R10.1, U2.1; no longer U2.6
- net at R7.1, R8.1: now also R9.1, U1.6; no longer U2.1
- net at R5.1: now also R1.2, R2.2, R4.1, R6.1, R7.2, R8.2, R9.2, R3.2; no longer U1.6
- net ATTN3out: now reaches U3.5
- net ATTN3out: now also U4.2; no longer C2.1
- net at R1.1, R2.1, U1.1: now also R3.1
- net ATTN1bp: now reaches U1.3, U1.4
- net ATTN1out: now reaches U1.5, U2.2
- net at R15.1, R17.2, R18.2: now also R10.2, R11.2, R12.2, R13.1, R14.1, R16.2; no longer R13.2, R14.2, R16.1
- net at R17.1, R18.1: now also R16.1, U2.6; no longer U3.6
- net ATTN2bp: now reaches U2.3, U2.4
- net ATTN2out: now reaches U2.5, U3.2
- net ATTN3bp: now reaches U3.3, U3.4
- new net: R28.1, R29.1, R30.1, U4.1
- new net: R34.1, R35.1, R36.1, U4.6
- new net: R19.2, R20.2, R21.2, R22.1, R23.1, R24.1, R25.2, R26.2, R27.2
- new net: R28.2, R29.2, R30.2, R31.1, R32.1, R33.1, R34.2, R35.2, R36.2
- new net: R25.1, R26.1, R27.1, U3.6
- new net: R19.1, R20.1, R21.1, U3.1
- new net ATTN4bp: U4.3, U4.4
- new net ATTN4out: C2.1, U4.5
Other:
- note added: "Attenuator #1 (-3db)"
- note added: "Attenuator #2 (-6db)"
- note added: "Attenuator #3(-12db)"
- note added: "Attenuator #4 (-24db)"
- note added: "PI Attenuator for A-RFID Cobbles"
- moved on the sheet: C1, Input1, Output1, R1, R2, R4, R6, U1
